Commit message: Added casterwheel and lidar integration for 2D map

File: urdf/robot.urdf (robot description, URDF)
Before this commit: robot diff_drive_bot, 3 links, 2 joints
Links:
- added link caster_wheel, mass 0.05; collision sphere radius=0.0375; visual sphere radius=0.0375
- added link lidar_link, mass 0.1
- added link lidar_mount, mass 0.1; collision cylinder length=0.04 radius=0.05; visual cylinder length=0.04 radius=0.05
Joints:
- added joint caster_wheel_joint: type fixed, parent base_link, child caster_wheel, origin xyz=0.23 0 0.0375 rpy=0 0 0
- added joint laser_joint: type fixed, parent base_link, child lidar_mount, origin xyz=-0.15 0 0.295 rpy=0 0 0
- added joint lidar_link_joint: type fixed, parent lidar_mount, child lidar_link, origin xyz=0 0 0.02 rpy=0 0 0
